File: hardware/NeoGeoController2USB.sch (KiCad schematic (older format))
At the start: 13 parts, among them CON1 AVR-ISP6, J1 USB, J2 DB15, U1 ATMEGA32U2-AU, X1 16Mhz

Commit message: Adding access to serial port. Fix controller pinout numering.
Parts:
- added CON2: TTL_6, ~, symbol TTL_6
- added R4, R5, R6: 22ohms, ~, symbol R
Connections:
- wire segments 70 -> 90
- no-connect marks 5 -> 4
Other:
- moved on the sheet: C3
